File: Hardware/v1.0.kicad_pcb (KiCad board)
At the start: 4 copper layers, 50.5 x 15 mm, 47 parts, among them J1 Conn_01x02_Pin, J2 Conn_01x01_Pin, J3 USB_C_Receptacle_PowerOnly_6P, J4 Conn_02x03_Odd_Even, J5 Conn_01x01_Pin, J6 Conn_01x01_Pin, J7 Conn_01x01_Pin, M1 Motor_DC, Q1 BSS138, U1 MCP73831-2-MC, U2 nRF52840, Y1 Crystal_Small

Commit message: Re-export all production files via KiCad 10 CLI
- KiCad source: updated PCB, schematic, project files
- Gerbers: switched from Protel to KiCad (.gbr) extensions
- Drill files: regenerated with gerber drill map
- STEP & GLB: re-exported 3D models
- Schematic PDF: re-exported
- Netlist: re-exported (kicad + XML)
- Gitignore: added tempfile exclusion
Parts:
- added J8: Conn_01x02_Pin, RF_Antenna:Texas_SWRA117D_2.4GHz_Left, F.Cu at (195.2, 49.9)
Connections:
- C18 pad 1: ANT -> Net-(J8-Pin_2)
Routing:
- net ANT: track 84.4 -> 0.00 mm, vias 2 -> 0
- net Net-(J8-Pin_2): track 0.00 -> 45.9 mm, vias 0 -> 1
Other:
- board size 50.5 x 15 mm -> 52.7 x 15 mm
